File: SparkFun_DB9_Breakout.kicad_sch (KiCad schematic)
At the start: 12 parts

Commit message: Renames DE9 footprint/symbol
Parts:
- added J1: A-DS 09 A/KG-T4S, footprints:CONN_A-DS 09 A&slash_KG-T4S_ASM, symbol 2025-03-10_17-10-03:A-DS_09_A_KG-T4S
Changed lines of the file:
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@@
+		)
+	)
+	(symbol
+		(lib_id "2025-03-10_17-10-03:A-DS_09_A_KG-T4S")
+		(at 133.35 100.33 0)
+		(unit 1)
+		(exclude_from_sim no)
+		(in_bom yes)
+		(on_board yes)
+		(dnp no)
+		(fields_autoplaced yes)
+		(property "Reference" "J1"
+			(at 138.43 97.7899 0)
+			(effects
+				(font
+					(size 1.524 1.524)
+				)
+				(justify left)
+			)
+		)
+		(property "Value" "A-DS 09 A/KG-T4S"
+			(at 138.43 100.3299 0)
+			(effects
+				(font
+					(size 1.524 1.524)
+				)
+				(justify left)
+			)
+		)
+		(property "Footprint" "footprints:CONN_A-DS 09 A&slash_KG-T4S_ASM"
+			(at 138.43 102.8699 0)
+			(effects
+				(font
+					(size 1.27 1.27)
+					(italic yes)
+				)
+				(justify left)
+			)
+		)
+		(property "Datasheet" "A-DS 09 A/KG-T4S"
+			(at 131.572 120.65 0)
+			(effects
+				(font
+					(size 1.27 1.27)
+					(italic yes)
+				)
+				(hide yes)
+			)
+		)
+		(property "Description" ""
+			(at 133.35 100.33 0)
+			(effects
+				(font
+					(size 1.27 1.27)
+				)
+				(hide yes)
+			)
+		)
+		(pin "5"
+		)
+		(pin "6"
+		)
+		(pin "1"
+		)
+		(pin "2"
+		)
+		(pin "7"
+		)
+		(pin "3"
+		)
+		(pin "8"
+		)
+		(pin "4"
+		)
+		(pin "9"
+		)
+		(instances
+			(project ""
+				(path "/e3dd3ae4-244d-4cba-9cca-5d2abf83f29a"
+					(reference "J1")
+					(unit 1)
+				)
+			)
 		)
 	)

Commit message: Fixes all symbols and footprint names
Parts:
- removed J1: A-DS 09 A/KG-T4S, footprints:CONN_A-DS 09 A&slash_KG-T4S_ASM, symbol 2025-03-10_17-10-03:A-DS_09_A_KG-T4S
- added J1: DE9-Male, footprints:CONN_A-DS 09 A&slash_KG-T4S_ASM, symbol 2025-03-10_17-10-03:DE9-Male
Changed lines of the file:
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@@
+	)
+	(symbol
+		(lib_id "2025-03-10_17-10-03:DE9-Male")
+		(at 132.08 105.41 0)
+		(unit 1)
+		(exclude_from_sim no)
+		(in_bom yes)
+		(on_board yes)
+		(dnp no)
+		(fields_autoplaced yes)
+		(property "Reference" "J1"
+			(at 137.16 101.5999 0)
+			(effects
+				(font
+					(size 1.524 1.524)
+				)
+				(justify left)
+			)
+		)
+		(property "Value" "DE9-Male"
+			(at 137.16 104.1399 0)
+			(effects
+				(font
+					(size 1.524 1.524)
+				)
+				(justify left)
+			)
+		)
+		(property "Footprint" "footprints:CONN_A-DS 09 A&slash_KG-T4S_ASM"
+			(at 137.16 106.6799 0)
+			(effects
+				(font
+					(size 1.27 1.27)
+					(italic yes)
+				)
+				(justify left)
+			)
+		)
+		(property "Datasheet" ""
+			(at 130.302 124.714 0)
+			(effects
+				(font
+					(size 1.27 1.27)
+					(italic yes)
+				)
+				(hide yes)
+			)
+		)
+		(property "Description" ""
+			(at 132.08 105.41 0)
+			(effects
+				(font
+					(size 1.27 1.27)
+				)
+				(hide yes)
+			)
+		)
+		(pin "9"
+		)
+		(pin "7"
+		)
+		(pin "6"
+		)
+		(pin "4"
+		)
+		(pin "2"
+		)
+		(pin "1"
+		)
+		(pin "8"
+		)
+		(pin "5"
+		)
+		(pin "3"
+		)
+		(instances
+			(project ""
+				(path "/e3dd3ae4-244d-4cba-9cca-5d2abf83f29a"
+					(reference "J1")
+					(unit 1)
+				)
+			)
+		)
 	)
 	(symbol
@@
 					(unit 1)
 				)
-			)
-		)
-	)
-	(symbol
-		(lib_id "2025-03-10_17-10-03:A-DS_09_A_KG-T4S")
-		(at 133.35 100.33 0)
-		(unit 1)
-		(exclude_from_sim no)
-		(in_bom yes)
-		(on_board yes)
-		(dnp no)
-		(fields_autoplaced yes)
-		(property "Reference" "J1"
-			(at 138.43 97.7899 0)
-			(effects
-				(font
-					(size 1.524 1.524)
-				)
-				(justify left)
-			)
-		)
-		(property "Value" "A-DS 09 A/KG-T4S"
-			(at 138.43 100.3299 0)
-			(effects
-				(font
-					(size 1.524 1.524)
-				)
-				(justify left)
-			)
-		)
-		(property "Footprint" "footprints:CONN_A-DS 09 A&slash_KG-T4S_ASM"
-			(at 138.43 102.8699 0)
-			(effects
-				(font
-					(size 1.27 1.27)
-					(italic yes)
-				)
-				(justify left)
-			)
-		)
-		(property "Datasheet" "A-DS 09 A/KG-T4S"
-			(at 131.572 120.65 0)
-			(effects
-				(font
-					(size 1.27 1.27)
-					(italic yes)
-				)
-				(hide yes)
-			)
-		)
-		(property "Description" ""
-			(at 133.35 100.33 0)
-			(effects
-				(font
-					(size 1.27 1.27)
-				)
-				(hide yes)
-			)
-		)
-		(pin "5"
-		)
-		(pin "6"
-		)
-		(pin "1"
-		)
-		(pin "2"
-		)
-		(pin "7"
-		)
-		(pin "3"
-		)
-		(pin "8"
-		)
-		(pin "4"
-		)
-		(pin "9"
-		)
-		(instances
-			(project ""
-				(path "/e3dd3ae4-244d-4cba-9cca-5d2abf83f29a"
-					(reference "J1")
-					(unit 1)
-				)

Commit message: Adds some nets, basic outline
Parts:
- removed J1: DE9-Male, footprints:CONN_A-DS 09 A&slash_KG-T4S_ASM, symbol 2025-03-10_17-10-03:DE9-Male
- removed ST3, ST4: Stand_off, SparkFun-Hardware:Standoff, symbol SparkFun-Hardware:Standoff
- added J1: DB9-Female, DB9_Footprint:DB9, symbol DB9-Female:DB9 Female
- added J2: Conn_01x09, SparkFun-Connector:1x09, symbol SparkFun-Connector:Conn_01x09
Connections:
- new net CTS: J1.7 (CTS), J2.6 (Pin_6)
- new net DCD: J1.1 (DCD), J2.1 (Pin_1)
- new net DSR: J1.6 (DSR), J2.5 (Pin_5)
- new net DTR: J1.4 (DTR), J2.4 (Pin_4)
- new net GND: J1.5 (GND), J2.9 (Pin_9)
- new net RI: J1.9 (RI), J2.8 (Pin_8)
- new net RTS: J1.8 (RTS), J2.7 (Pin_7)
- new net RXD: J1.3 (RXD), J2.3 (Pin_3)
- new net TXD: J1.2 (TXD), J2.2 (Pin_2)
