File: Female/SparkFun_DE9_Female_Breakout.kicad_sch (KiCad schematic)
At the start: 9 parts, among them J1 DE9-Female, J2 Conn_01x09, J3 Conn_01x01, J4 Conn_01x01

Commit message: Fixes common pinouts tables in schematics
Other:
- note added: "RS232 + RS485 Pinout Male"
- note removed: "RS232 + RS485 Pinout Female"
Changed lines of the file:
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@@
 		)
 	)
-	(text "RS232 + RS485 Pinout Female"
+	(text "RS232 + RS485 Pinout Male"
 		(exclude_from_sim no)
-		(at 195.58 72.39 0)
+		(at 194.31 71.12 0)
 		(effects
 			(font
@@
 	(wire
 		(pts
+			(xy 87.63 97.79) (xy 74.93 97.79)
+		)
+		(stroke
+			(width 0)
+			(type default)
+		)
+	)
+	(wire
+		(pts
 			(xy 69.85 95.25) (xy 74.93 95.25)
-		)
-		(stroke
-			(width 0)
-			(type default)
-		)
-	)
-	(wire
-		(pts
-			(xy 87.63 97.79) (xy 74.93 97.79)
 		)
 		(stroke
@@
 			(table_cell "Pin 1"
 				(exclude_from_sim no)
-				(at 180.594 74.168 0)
+				(at 180.34 72.39 0)
+				(size 7.62 2.54)
+				(margins 0.9525 0.9525 0.9525 0.9525)
+				(span 1 1)
+				(fill
+					(type none)
+				)
+				(effects
+					(font
+						(size 1.27 1.27)
+					)
+					(justify left top)
+				)
+			)
+			(table_cell "Data Carrier Detect (DCD) "
+				(exclude_from_sim no)
+				(at 187.96 72.39 0)
+				(size 31.75 2.54)
+				(margins 0.9525 0.9525 0.9525 0.9525)
+				(span 1 1)
+				(fill
+					(type none)
+				)
+				(effects
+					(font
+						(size 1.27 1.27)
+					)
+					(justify left top)
+				)
+			)
+			(table_cell "Pin 2"
+				(exclude_from_sim no)
+				(at 180.34 74.93 0)
+				(size 7.62 2.54)
+				(margins 0.9525 0.9525 0.9525 0.9525)
+				(span 1 1)
+				(fill
+					(type none)
+				)
+				(effects
+					(font
+						(size 1.27 1.27)
+					)
+					(justify left top)
+				)
+			)
+			(table_cell "Received Data (RXD) "
+				(exclude_from_sim no)
+				(at 187.96 74.93 0)
+				(size 31.75 2.54)
+				(margins 0.9525 0.9525 0.9525 0.9525)
+				(span 1 1)
+				(fill
+					(type none)
+				)
+				(effects
+					(font
+						(size 1.27 1.27)
+					)
+					(justify left top)
+				)
+			)
+			(table_cell "Pin 3"
+				(exclude_from_sim no)
+				(at 180.34 77.47 0)
+				(size 7.62 2.54)
+				(margins 0.9525 0.9525 0.9525 0.9525)
+				(span 1 1)
+				(fill
+					(type none)
+				)
+				(effects
+					(font
+						(size 1.27 1.27)
+					)
+					(justify left top)
+				)
+			)
+			(table_cell "Transmit Data (TXD) "
+				(exclude_from_sim no)
+				(at 187.96 77.47 0)
+				(size 31.75 2.54)
+				(margins 0.9525 0.9525 0.9525 0.9525)
+				(span 1 1)
+				(fill
+					(type none)
+				)
+				(effects
+					(font
+						(size 1.27 1.27)
+					)
+					(justify left top)
+				)
+			)
+			(table_cell "Pin 4"
+				(exclude_from_sim no)
+				(at 180.34 80.01 0)
+				(size 7.62 2.54)
+				(margins 0.9525 0.9525 0.9525 0.9525)
+				(span 1 1)
+				(fill
+					(type none)
+				)
+				(effects
+					(font
+						(size 1.27 1.27)
+					)
+					(justify left top)
+				)
+			)
+			(table_cell "Data Terminal Ready (DTR) "
+				(exclude_from_sim no)
+				(at 187.96 80.01 0)
+				(size 31.75 2.54)
+				(margins 0.9525 0.9525 0.9525 0.9525)
+				(span 1 1)
+				(fill
+					(type none)
+				)
+				(effects
+					(font
+						(size 1.27 1.27)
+					)
+					(justify left top)
+				)
+			)
+			(table_cell "Pin 5"
+				(exclude_from_sim no)
+				(at 180.34 82.55 0)
 				(size 7.62 2.54)
 				(margins 0.9525 0.9525 0.9525 0.9525)
@@
 			(table_cell "Ground (GND)"
 				(exclude_from_sim no)
-				(at 188.214 74.168 0)
-				(size 31.75 2.54)
-				(margins 0.9525 0.9525 0.9525 0.9525)
-				(span 1 1)
-				(fill
-					(type none)
-				)
-				(effects
-					(font
-						(size 1.27 1.27)
-					)
-					(justify left top)
-				)
-			)
-			(table_cell "Pin 2"
-				(exclude_from_sim no)
-				(at 180.594 76.708 0)
-				(size 7.62 2.54)
-				(margins 0.9525 0.9525 0.9525 0.9525)
-				(span 1 1)
-				(fill
-					(type none)
-				)
-				(effects
-					(font
-						(size 1.27 1.27)
-					)
-					(justify left top)
-				)
-			)
-			(table_cell "Data Terminal Ready (DTR)"
-				(exclude_from_sim no)
-				(at 188.214 76.708 0)
-				(size 31.75 2.54)
-				(margins 0.9525 0.9525 0.9525 0.9525)
-				(span 1 1)
-				(fill
-					(type none)
-				)
-				(effects
-					(font
-						(size 1.27 1.27)
-					)
-					(justify left top)
-				)
-			)
-			(table_cell "Pin 3"
-				(exclude_from_sim no)
-				(at 180.594 79.248 0)
-				(size 7.62 2.54)
-				(margins 0.9525 0.9525 0.9525 0.9525)
-				(span 1 1)
-				(fill
-					(type none)
-				)
-				(effects
-					(font
-						(size 1.27 1.27)
-					)
-					(justify left top)
-				)
-			)
-			(table_cell "Received Data (RXD)"
-				(exclude_from_sim no)
-				(at 188.214 79.248 0)
-				(size 31.75 2.54)
-				(margins 0.9525 0.9525 0.9525 0.9525)
-				(span 1 1)
-				(fill
-					(type none)
-				)
-				(effects
-					(font
-						(size 1.27 1.27)
-					)
-					(justify left top)
-				)
-			)
-			(table_cell "Pin 4"
-				(exclude_from_sim no)
-				(at 180.594 81.788 0)
-				(size 7.62 2.54)
-				(margins 0.9525 0.9525 0.9525 0.9525)
-				(span 1 1)
-				(fill
-					(type none)
-				)
-				(effects
-					(font
-						(size 1.27 1.27)
-					)
-					(justify left top)
-				)
-			)
-			(table_cell "Transmit (TXD)"
-				(exclude_from_sim no)
-				(at 188.214 81.788 0)
-				(size 31.75 2.54)
-				(margins 0.9525 0.9525 0.9525 0.9525)
-				(span 1 1)
-				(fill
-					(type none)
-				)
-				(effects
-					(font
-						(size 1.27 1.27)
-					)
-					(justify left top)
-				)
-			)
-			(table_cell "Pin 5"
-				(exclude_from_sim no)
-				(at 180.594 84.328 0)
-				(size 7.62 2.54)
-				(margins 0.9525 0.9525 0.9525 0.9525)
-				(span 1 1)
-				(fill
-					(type none)
-				)
-				(effects
-					(font
-						(size 1.27 1.27)
-					)
-					(justify left top)
-				)
-			)
-			(table_cell "Data Carrier Detect (DCD)"
-				(exclude_from_sim no)
-				(at 188.214 84.328 0)
+				(at 187.96 82.55 0)
 				(size 31.75 2.54)
 				(margins 0.9525 0.9525 0.9525 0.9525)
@@
 			(table_cell "Pin 6"
 				(exclude_from_sim no)
-				(at 180.594 86.868 0)
-				(size 7.62 2.54)
-				(margins 0.9525 0.9525 0.9525 0.9525)
-				(span 1 1)
-				(fill
-					(type none)
-				)
-				(effects
-					(font
-						(size 1.27 1.27)
-					)
-					(justify left top)
-				)
-			)
-			(table_cell "Ring Indicator (RI)"
-				(exclude_from_sim no)
-				(at 188.214 86.868 0)
+				(at 180.34 85.09 0)
+				(size 7.62 2.54)
+				(margins 0.9525 0.9525 0.9525 0.9525)
+				(span 1 1)
+				(fill
+					(type none)
+				)
+				(effects
+					(font
+						(size 1.27 1.27)
+					)
+					(justify left top)
+				)
+			)
+			(table_cell "Request to send (RTS) "
+				(exclude_from_sim no)
+				(at 187.96 85.09 0)
 				(size 31.75 2.54)
 				(margins 0.9525 0.9525 0.9525 0.9525)
@@
 			(table_cell "Pin 7"
 				(exclude_from_sim no)
-				(at 180.594 89.408 0)
-				(size 7.62 2.54)
-				(margins 0.9525 0.9525 0.9525 0.9525)
-				(span 1 1)
-				(fill
-					(type none)
-				)
-				(effects
-					(font
-						(size 1.27 1.27)
-					)
-					(justify left top)
-				)
-			)
-			(table_cell "Ready to Send (RTS)"
-				(exclude_from_sim no)
-				(at 188.214 89.408 0)
+				(at 180.34 87.63 0)
+				(size 7.62 2.54)
+				(margins 0.9525 0.9525 0.9525 0.9525)
+				(span 1 1)
+				(fill
+					(type none)
+				)
+				(effects
+					(font
+						(size 1.27 1.27)
+					)
+					(justify left top)
+				)
+			)
+			(table_cell "Request to send (RTS) "
+				(exclude_from_sim no)
+				(at 187.96 87.63 0)
 				(size 31.75 2.54)
 				(margins 0.9525 0.9525 0.9525 0.9525)
@@
 			(table_cell "Pin 8"
 				(exclude_from_sim no)
-				(at 180.594 91.948 0)
-				(size 7.62 2.54)
-				(margins 0.9525 0.9525 0.9525 0.9525)
-				(span 1 1)
-				(fill
-					(type none)
-				)
-				(effects
-					(font
-						(size 1.27 1.27)
-					)
-					(justify left top)
-				)
-			)
-			(table_cell "Clear to Send (CTS)"
-				(exclude_from_sim no)
-				(at 188.214 91.948 0)
+				(at 180.34 90.17 0)
+				(size 7.62 2.54)
+				(margins 0.9525 0.9525 0.9525 0.9525)
+				(span 1 1)
+				(fill
+					(type none)
+				)
+				(effects
+					(font
+						(size 1.27 1.27)
+					)
+					(justify left top)
+				)
+			)
+			(table_cell "Clear to Send (CTS) "
+				(exclude_from_sim no)
+				(at 187.96 90.17 0)
 				(size 31.75 2.54)
 				(margins 0.9525 0.9525 0.9525 0.9525)
@@
 			(table_cell "Pin 9"
 				(exclude_from_sim no)
-				(at 180.594 94.488 0)
-				(size 7.62 2.54)
-				(margins 0.9525 0.9525 0.9525 0.9525)
-				(span 1 1)
-				(fill
-					(type none)
-				)
-				(effects
-					(font
-						(size 1.27 1.27)
-					)
-					(justify left top)
-				)
-			)
-			(table_cell "Data Set Ready (DSR)"
-				(exclude_from_sim no)
-				(at 188.214 94.488 0)
-				(size 31.75 2.54)
-				(margins 0.9525 0.9525 0.9525 0.9525)
+				(at 180.34 92.71 0)
+				(size 7.62 2.54)
+				(margins 0.9525 0.9525 0.9525 0.9525)
+				(span 1 1)
+				(fill
+					(type none)
+				)
+				(effects
+					(font
+						(size 1.27 1.27)
+					)
+					(justify left top)
+				)
+			)
+			(table_cell "Ring Indicator (RI) "
+				(exclude_from_sim no)
+				(at 187.96 92.71 0)
+				(size 31.75 2.54)
+				(margins 0.9525 0.9525 0.9525 0.9525)
