File: Hardware/Female/SparkFun_DE9_Female_Breakout.kicad_sch (KiCad schematic)
At the start: 9 parts, among them J1 Conn_01x01, J2 Conn_01x09, J4 Conn_01x01, J5 DE9-Male

Commit message: Removes the local symbols/footprints, moves designs to Hardware folder
Parts:
- removed J1: Conn_01x01, SparkFun-Connector:1x01, symbol SparkFun-Connector:Conn_01x01
- removed J5: DE9-Male, DE9-Footprint:DE9, symbol DE9-Male:DE9-Male
- added J1: DE9 Female, SparkFun-Connector:DE9_Female, symbol SparkFun-Connector:DE9_Female
- added J3: Conn_01x01, SparkFun-Connector:1x01, symbol SparkFun-Connector:Conn_01x01
Connections:
- net 1: now also J1.1
- net 2: now also J1.2
- net 3: now also J1.3
- net 4: now also J1.4
- net 5: now also J1.5
- net 6: now also J1.6
- net 7: now also J1.7
- net 8: now also J1.8
- net 9: now also J1.9
- net GND: now also J3.1 (Pin_1)
Other:
- note added: "D-Sub Female Connector - DE9"
- note added: "RS232 + RS485 Pinout Male"
- note removed: "D-Sub Male Connector - DE9"
- note removed: "RS232 + RS485 Pinout Female"
- moved on the sheet: J2
