File: Hardware/Female/SparkFun_DE9_Female_Breakout.kicad_sch (KiCad schematic)
At the start: 9 parts, among them J1 DE9 Female, J2 Conn_01x09, J3 Conn_01x01, J4 Conn_01x01

Commit message: Fix pin layout
Adds model for female socket
FIxes male footprint and symbol; updates schematic and PCB
Parts:
- J1: footprint SparkFun-Connector:DE9_Female -> SparkFun-Connector:DE9_Socket_Horizontal_PTH
