File: Hardware/Male/SparkFun_DE9_Male_Breakout.kicad_pcb (KiCad board)
At the start: 2 copper layers, 22.9 x 31.8 mm, 43 parts, among them J1 Conn_01x01, J2 Conn_01x09, J3 DE9 Male, J4 Conn_01x01

Commit message: Fixes silk and pinout on DE9 connector
Parts:
- J3: value DE9 Male -> DE9 Header; footprint SparkFun-Connector:DE9_Male -> SparkFun-Connector:DE9_Header_Horizontal_PTH
- moved kibuzzard-67D496F6 20.3 mm to (135.3, 118.7)
- moved J2 20.3 mm to (137.2, 98.4), turned to -90 degrees
- moved kibuzzard-67D496EA 15.2 mm to (135.3, 116.2)
- moved kibuzzard-67DDA3B0 12.7 mm to (135.3, 118.7)
- moved kibuzzard-67DDA3B8 12.7 mm to (135.3, 116.2)
- moved kibuzzard-67DDA3D5 12.7 mm to (135.3, 113.7)
- moved kibuzzard-67DDA3E0 12.7 mm to (135.3, 111.1)
- moved kibuzzard-67D49687 10.2 mm to (135.3, 108.6)
- moved kibuzzard-67D496C7 10.2 mm to (135.3, 103.5)
- moved kibuzzard-67D496E4 10.2 mm to (135.3, 113.7)
- moved kibuzzard-67DDA399 10.2 mm to (135.3, 103.5)
- moved kibuzzard-67F7FDBF 10.2 mm to (135.3, 108.6)
- moved kibuzzard-67D496B8 10.2 mm to (135.3, 106.0)
- moved kibuzzard-67D496CD 10.2 mm to (135.3, 101.0)
- moved kibuzzard-67D496D5 10.2 mm to (135.3, 98.4)
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Connections:
- J2 pad 1: /1 -> /5
- J2 pad 2: /2 -> /4
- J2 pad 4: /4 -> /2
- J2 pad 5: /5 -> /1
- J2 pad 6: /6 -> /9
- J2 pad 7: /7 -> /8
- J2 pad 8: /8 -> /7
- J2 pad 9: /9 -> /6
Other:
- board text added: "v11"
- board text removed: "v10"
