File: Hardware/Male/SparkFun_DE9_Male_Breakout.kicad_pcb (KiCad board)
At the start: 2 copper layers, 22.9 x 31.8 mm, 43 parts, among them J1 Conn_01x01, J2 Conn_01x09, J3 DE9 Header, J4 Conn_01x01

Commit message: Fix pin layout
Adds model for female socket
FIxes male footprint and symbol; updates schematic and PCB
Parts:
- moved kibuzzard-67DDBDCA 10.8 mm to (128.6, 103.2)
- moved kibuzzard-67DDBDD7 10.8 mm to (128.5, 114.0)
- moved kibuzzard-67D49687 10.2 mm to (135.3, 98.4)
- moved kibuzzard-67D496D5 10.2 mm to (135.3, 108.6)
- moved kibuzzard-67DDA3AA 10.2 mm to (135.3, 108.6)
- moved kibuzzard-67F7FDBF 10.2 mm to (135.3, 98.4)
- moved kibuzzard-67DDBDDC 8.26 mm to (121.5, 112.7)
- moved kibuzzard-67DDBDFC 8.26 mm to (121.6, 104.5)
- moved kibuzzard-67DDA3B0 7.62 mm to (135.3, 111.1)
- moved kibuzzard-67DDA3E0 7.62 mm to (135.3, 118.7)
- moved kibuzzard-67DDBDB0 5.71 mm to (128.5, 105.7)
- moved kibuzzard-67DDBDD2 5.71 mm to (128.6, 111.4)
- moved kibuzzard-67D496B8 5.08 mm to (135.3, 101.0)
- moved kibuzzard-67D496CD 5.08 mm to (135.3, 106.0)
- moved kibuzzard-67DDA391 5.08 mm to (135.3, 101.0)
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Connections:
- net /3 renamed Net-(J2-Pin_3)
- J2 pad 1: /5 -> Net-(J2-Pin_1)
- J2 pad 2: /4 -> Net-(J2-Pin_2)
- J2 pad 4: /2 -> Net-(J2-Pin_4)
- J2 pad 5: /1 -> Net-(J2-Pin_5)
- J2 pad 6: /9 -> Net-(J2-Pin_6)
- J2 pad 7: /8 -> Net-(J2-Pin_7)
- J2 pad 8: /7 -> Net-(J2-Pin_8)
- J2 pad 9: /6 -> Net-(J2-Pin_9)
- J3 pad 1: /1 -> Net-(J2-Pin_1)
- J3 pad 2: /2 -> Net-(J2-Pin_2)
- J3 pad 4: /4 -> Net-(J2-Pin_4)
- J3 pad 5: /5 -> Net-(J2-Pin_5)
- J3 pad 6: /6 -> Net-(J2-Pin_6)
- J3 pad 7: /7 -> Net-(J2-Pin_7)
- J3 pad 8: /8 -> Net-(J2-Pin_8)
- J3 pad 9: /9 -> Net-(J2-Pin_9)
Routing:
- net Net-(J2-Pin_6): track 0.00 -> 16.2 mm
- net /9: track 16.2 -> 0.00 mm
- net Net-(J2-Pin_7): track 0.00 -> 16.1 mm
- net /8: track 16.1 -> 0.00 mm
- net Net-(J2-Pin_8): track 0.00 -> 16.0 mm
- net /7: track 16.0 -> 0.00 mm
- net Net-(J2-Pin_9): track 0.00 -> 15.9 mm
- net /6: track 15.9 -> 0.00 mm
- net Net-(J2-Pin_5): track 0.00 -> 13.0 mm
- net /1: track 13.0 -> 0.00 mm
- net Net-(J2-Pin_4): track 0.00 -> 12.9 mm
- net /2: track 12.9 -> 0.00 mm
- net Net-(J2-Pin_2): track 0.00 -> 12.7 mm
- net /4: track 12.7 -> 0.00 mm
- net Net-(J2-Pin_1): track 0.00 -> 12.6 mm
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